File: Examples/Eagle/Simple_BRD/Simple_BRD.brd (EAGLE design)
At the start: 61 x 64.8 mm, 16 parts

Commit message: Added support for test point output
Parts:
- added E$13: (no value), testpad:B1,27
- added E$14: (no value), testpad:B2,54
- added E$15: (no value), testpad:P1-13
- added E$16: (no value), testpad:P1-13Y
- added E$17: (no value), testpad:P1-17
- added E$18: (no value), testpad:P1-17Y
- added E$19: (no value), testpad:P1-20
- added E$24: (no value), testpad:P1-20Y
- added E$25: (no value), testpad:P2-38-17
- added E$26: (no value), testpad:P2-38-20
- added E$27: (no value), testpad:P5-25-13
- added E$28: (no value), testpad:P5-25-17
- added E$29: (no value), testpad:TP06R
- added E$30: (no value), testpad:TP06SQ
- added E$31: (no value), testpad:TP07R
- added E$32: (no value), testpad:TP07SQ
- added E$33: (no value), testpad:TP08R
- added E$34: (no value), testpad:TP08SQ
- added E$35: (no value), testpad:TP09R
- added E$36: (no value), testpad:TP09SQ
- added E$37: (no value), testpad:TP10R
- added E$38: (no value), testpad:TP10SQ
- added E$39: (no value), testpad:TP11R
- added E$40: (no value), testpad:TP11SQ
- added E$41: (no value), testpad:TP12R
- added E$42: (no value), testpad:TP12SQ
- added E$43: (no value), testpad:TP13R
- added E$44: (no value), testpad:TP13SQ
- added E$45: (no value), testpad:TP14R
- added E$46: (no value), testpad:TP14SQ
- added E$47: (no value), testpad:TP15R
- added E$48: (no value), testpad:TP15SQ
- added E$49: (no value), testpad:TP16R
- added E$50: (no value), testpad:TP16SQ
- added E$51: (no value), testpad:TP17R
- added E$52: (no value), testpad:TP17SQ
- added E$53: (no value), testpad:TP18R
- added E$54: (no value), testpad:TP18SQ
- added E$55: (no value), testpad:TP19R
- added E$56: (no value), testpad:TP19SQ
- added E$57: (no value), testpad:TP20R
- added E$58: (no value), testpad:TP20SQ
Other:
- board size 61 x 64.8 mm -> 82.5 x 67.3 mm
